File: pcb/optionrom.sch (KiCad schematic (older format))
At the start: 6 parts, among them P1 CONN_01X02, U1 CAT24C32

Commit message: allow STM32 to control option-ROM WP pin.
Parts:
- removed P1: CONN_01X02, Pin_Headers:Pin_Header_Straight_1x02, symbol CONN_01X02
Connections:
- net WP: now reaches R1.2, U1.7 (WP)
Other:
- note removed: "Write Enable"
Changed lines of the file:
@@
-	1    0    0    -1
-$EndComp
-$Comp
-L CONN_01X02 P1
-U 1 1 57B302AE
-P 5700 4050
-F 0 "P1" H 5700 4200 50  0000 C CNN
-F 1 "CONN_01X02" V 5800 4050 50  0000 C CNN
-F 2 "Pin_Headers:Pin_Header_Straight_1x02" H 5700 4050 50  0001 C CNN
-F 3 "" H 5700 4050 50  0000 C CNN
-	1    5700 4050
 	1    0    0    -1
 $EndComp
@@
 Connection ~ 5500 3400
 Wire Wire Line
-	5500 4300 5500 4100
-Wire Wire Line
-	3100 4300 5500 4300
-Wire Wire Line
 	4600 4300 4600 4000
 Connection ~ 4600 4300
-Text Notes 5950 4050 0    60   ~ 0
-Write Enable
 Wire Wire Line
 	3100 2800 5900 2800
@@
 Text HLabel 3100 2800 0    60   Input ~ 0
 PIVCC
+Wire Wire Line
+	3100 4300 4600 4300
+Text HLabel 6900 4000 2    60   Input ~ 0
+WP
+Wire Wire Line
+	5500 4000 6900 4000
 $EndSCHEMATC

Commit message: added SPI flash and connections for STM32 to control the sensors
Parts:
- added P8: CONN_01X02, Pin_Headers:Pin_Header_Straight_1x02, symbol CONN_01X02
Connections:
- net GND: now also P8.2 (P2)
- net WP: no longer names the net of R1.2, U1.7 (WP)
- net WP: now also P8.1 (P1)
Changed lines of the file:
@@
 PIVCC
 Wire Wire Line
-	3100 4300 4600 4300
-Text HLabel 6900 4000 2    60   Input ~ 0
-WP
+	3100 4300 5500 4300
+$Comp
+L CONN_01X02 P8
+U 1 1 57B5BABB
+P 5700 4050
+F 0 "P8" H 5700 4200 50  0000 C CNN
+F 1 "CONN_01X02" V 5800 4050 50  0000 C CNN
+F 2 "Pin_Headers:Pin_Header_Straight_1x02" H 5700 4050 50  0001 C CNN
+F 3 "" H 5700 4050 50  0000 C CNN
+	1    5700 4050
+	1    0    0    -1
+$EndComp
 Wire Wire Line
-	5500 4000 6900 4000
+	5500 4300 5500 4100
 $EndSCHEMATC
